File: carte_robo_pince/carte_robo_pince.kicad_sch (KiCad schematic)
At the start: 9 parts, among them J1 Conn_01x18_Pin, J2 Conn_01x18_Pin, J3 Conn_01x03_Socket, J4 Conn_01x03_Socket, J5 Conn_01x03_Socket, J6 Conn_01x03_Socket, J7 Conn_01x03_Socket, J8 Conn_01x05_Socket

Commit message: pcb done
Parts:
- removed J8: Conn_01x05_Socket, Connector_PinSocket_2.54mm:PinSocket_1x05_P2.54mm_Vertical, symbol Connector:Conn_01x05_Socket
- added C1, C2: 100n, symbol GW_Passives:C_Small
Connections:
- net at BT1.1 (+), J3.2 (Pin_2), J4.2 (Pin_2)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: now also J6.2 (Pin_2)
- net +3.3V: now reaches J1.16 (Pin_16)
- net +3.3V: now also C1.1
- net +5V: now reaches J1.17 (Pin_17)
- net +5V: now also C2.1
- net at J1.18 (Pin_18): now also C1.2, C2.2
- no-connect marks 27 -> 24

Commit message: last update
Parts:
- BT1: footprint (none) -> Connector_PinHeader_2.54mm:PinHeader_1x02_P2.54mm_Vertical
- C1, C2: footprint (none) -> Capacitor_THT:C_Disc_D4.3mm_W1.9mm_P5.00mm
Connections:
- net GND: now also C1.2, C2.2, J1.18 (Pin_18)
Changed lines of the file:
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@@
+	(wire
+		(pts
+			(xy 73.66 111.76) (xy 73.66 115.57)
+		)
+		(stroke
+			(width 0)
+			(type default)
+		)
+	)
 	(wire
 		(pts
@@
 		(on_board yes)
 		(dnp no)
-		(fields_autoplaced yes)
 		(property "Reference" "J2"
-			(at 107.315 50.8 0)
+			(at 106.934 53.34 0)
 			(effects
 				(font
@@
 				(path "/89b969ca-cc58-4060-8a32-812d2d7c047c"
 					(reference "J7")
+					(unit 1)
+				)
+			)
+		)
+	)
+	(symbol
+		(lib_id "power:GND")
+		(at 73.66 115.57 0)
+		(unit 1)
+		(exclude_from_sim no)
+		(in_bom yes)
+		(on_board yes)
+		(dnp no)
+		(fields_autoplaced yes)
+		(property "Reference" "#PWR02"
+			(at 73.66 121.92 0)
+			(effects
+				(font
+					(size 1.27 1.27)
+				)
+				(hide yes)
+			)
+		)
+		(property "Value" "GND"
+			(at 73.66 120.65 0)
+			(effects
+				(font
+					(size 1.27 1.27)
+				)
+			)
+		)
+		(property "Footprint" ""
+			(at 73.66 115.57 0)
+			(effects
+				(font
+					(size 1.27 1.27)
+				)
+				(hide yes)
+			)
+		)
+		(property "Datasheet" ""
+			(at 73.66 115.57 0)
+			(effects
+				(font
+					(size 1.27 1.27)
+				)
+				(hide yes)
+			)
+		)
+		(property "Description" "Power symbol creates a global label with name \"GND\" , ground"
+			(at 73.66 115.57 0)
+			(effects
+				(font
+					(size 1.27 1.27)
+				)
+				(hide yes)
+			)
+		)
+		(pin "1"
+		)
+		(instances
+			(project "carte_robo_pince"
+				(path "/89b969ca-cc58-4060-8a32-812d2d7c047c"
+					(reference "#PWR02")
 					(unit 1)
 				)
@@
 			)
 		)
-		(property "Footprint" ""
+		(property "Footprint" "Capacitor_THT:C_Disc_D4.3mm_W1.9mm_P5.00mm"
 			(at 73.66 105.41 0)
 			(effects
@@
 			)
 		)
-		(property "Footprint" ""
+		(property "Footprint" "Connector_PinHeader_2.54mm:PinHeader_1x02_P2.54mm_Vertical"
 			(at 150.114 39.37 90)
 			(effects
@@
 			)
 		)
-		(property "Footprint" ""
+		(property "Footprint" "Capacitor_THT:C_Disc_D4.3mm_W1.9mm_P5.00mm"
 			(at 66.04 105.41 0)
 			(effects

Commit message: version
Parts:
- added C4: 1000u, Capacitor_THT:CP_Radial_D12.5mm_P5.00mm, symbol GW_Passives:C_Small
Connections:
- net +5V: now also BT1.1 (+), J3.2 (Pin_2), J4.2 (Pin_2), J5.2 (Pin_2), J6.2 (Pin_2), J7.2 (Pin_2), C4.2
- net GND: now also C4.1
Other:
- moved on the sheet: BT1
