File: carte_robo_pince/carte_robo_pince.kicad_pcb (KiCad board)
At the start: 2 copper layers, 45 x 50.5 mm, 10 parts, among them J1 Conn_01x18_Pin, J2 Conn_01x18_Pin, J3 Conn_01x03_Socket, J4 Conn_01x03_Socket, J5 Conn_01x03_Socket, J6 Conn_01x03_Socket, J7 Conn_01x03_Socket

Commit message: version
Parts:
- added C4: 1000u, Capacitor_THT:CP_Radial_D12.5mm_P5.00mm, F.Cu at (100.7, 108.9)
Connections:
- BT1 pad 1: Net-(BT1-+) -> /+5V
- J3 pad 2: Net-(BT1-+) -> /+5V
- J4 pad 2: Net-(BT1-+) -> /+5V
- J5 pad 2: Net-(BT1-+) -> /+5V
- J6 pad 2: Net-(BT1-+) -> /+5V
- J7 pad 2: Net-(BT1-+) -> /+5V
Routing:
- net /+5V: track 3.06 -> 53.9 mm
- net Net-(BT1-+): track 23.0 -> 0.00 mm
Other:
- board size 45 x 50.5 mm -> 52 x 50.7 mm
- board text added: "+"
- board text added: "GND"
- board text added: "M1"
- board text added: "M2"
- board text added: "M3"
- board text added: "M4"
- board text added: "M5"

Commit message: 19/03
Parts:
- added C3: 0.33pF, Capacitor_THT:C_Disc_D3.0mm_W1.6mm_P2.50mm, F.Cu at (97.0, 103.3)
- added C5: 0.1uF, Capacitor_THT:C_Disc_D3.0mm_W1.6mm_P2.50mm, F.Cu at (102.1, 103.3)
- added D1: LED, LED_THT:LED_D3.0mm, F.Cu at (97.5, 76.3)
- added R1: 330, Resistor_THT:R_Axial_DIN0207_L6.3mm_D2.5mm_P10.16mm_Horizontal, F.Cu at (103.7, 72.8)
- added U1: KA78M05_TO252, Package_TO_SOT_THT:TO-220-3_Horizontal_TabDown, F.Cu at (97.1, 100.7)
- BT1: value +5V -> +8V
- moved C4 7.08 mm to (101.4, 115.9)
- moved J7 5.04 mm to (113.2, 95.6)
- moved J6 4.90 mm to (113.2, 90.9)
- moved J3 1.97 mm to (113.1, 76.3)
- moved J5 1.88 mm to (113.2, 86.2)
- moved J4 1.87 mm to (113.1, 81.4)
- moved BT1 1.82 mm to (110.5, 100.2)
Connections:
- BT1 pad 1: /+5V -> /+8V
Routing:
- net /15_S4: track 49.2 -> 35.5 mm
- net /+5V: track 53.9 -> 64.9 mm
- net Net-(D1-A): track 0.00 -> 5.10 mm
- net /16_S0: track 39.1 -> 36.0 mm
- net /13_S2: track 14.7 -> 12.0 mm
- net /14_S3: track 14.6 -> 11.9 mm
- net Net-(U1-VI): track 0.00 -> 2.63 mm
- net /4_S5: track 40.4 -> 39.6 mm

Commit message: 01/04/25
Parts:
- added C6: 10u, Capacitor_THT:C_Disc_D3.0mm_W1.6mm_P2.50mm, F.Cu at (90.5, 87.1)
- added C7: 0.1u, Capacitor_THT:C_Disc_D3.0mm_W1.6mm_P2.50mm, F.Cu at (90.5, 84.8)
- added R2: 0.01, GW_Passives:R_2512_6332Metric, F.Cu at (86.9, 90.2)
- added R3: 3.3k, Resistor_THT:R_Axial_DIN0207_L6.3mm_D2.5mm_P10.16mm_Horizontal, F.Cu at (90.7, 72.2)
- added R4: 3.3k, Resistor_THT:R_Axial_DIN0207_L6.3mm_D2.5mm_P10.16mm_Horizontal, F.Cu at (87.5, 72.2)
- added SW1: SW_DIP_x01, Button_Switch_THT:SW_slide-03_P5_THT, F.Cu at (88.5, 107.0)
- added U2: INA219AxDCN, Package_TO_SOT_SMD:SOT-23-8, F.Cu at (87.6, 85.8)
- moved BT1 28.4 mm to (88.4, 118.1)
- moved R1 3.33 mm to (100.4, 72.3)
Connections:
- J1 pad 1: unconnected-(J1-Pin_1-Pad1) -> /SDA
- J2 pad 10: unconnected-(J2-Pin_10-Pad10) -> /SCL
- J7 pad 2: /+5V -> Net-(J7-Pin_2)
Routing:
- net /SCL: track 0.00 -> 63.8 mm, vias 0 -> 2
- net /+5V: track 64.9 -> 110.1 mm
- net Net-(J7-Pin_2): track 0.00 -> 37.8 mm
- net /SDA: track 0.00 -> 36.5 mm
- net Net-(U1-VI): track 2.63 -> 12.7 mm
- net /+8V: track 0.00 -> 6.14 mm
- net GND: track 0.00 -> 5.83 mm, vias 0 -> 2
- net /16_S0: track 36.0 -> 34.1 mm
- net Net-(D1-A): track 5.10 -> 4.21 mm
Other:
- board size 52 x 50.7 mm -> 62.7 x 50.7 mm
