File: carte_robo_main/Carte_main.kicad_pcb (KiCad board)
At the start: 2 copper layers, 45 x 50.5 mm, 13 parts, among them J1 Conn_01x18_Pin, J2 Conn_01x18_Pin, J3 Conn_01x02_Socket, J4 Conn_01x05_Socket

Commit message: last update
Parts:
- added R5: 100k, Resistor_THT:R_Axial_DIN0207_L6.3mm_D2.5mm_P10.16mm_Horizontal, F.Cu at (123.1, 74.1)
- added SW1: SW_Push, Button_Switch_THT:SW_PUSH_6mm_H5mm, F.Cu at (118.3, 83.8)
- moved J3 5.69 mm to (124.6, 90.4), turned to 180 degrees
- moved C1 3.13 mm to (130.7, 111.2)
- moved C2 3.13 mm to (130.7, 95.7)
- moved C3 3.13 mm to (130.7, 101.3)
- moved C4 3.13 mm to (130.7, 119.3)
- moved C5 3.13 mm to (130.7, 116.8)
- moved J1 3.13 mm to (133.6, 78.7)
- moved J2 3.13 mm to (156.4, 78.7)
- moved J4 3.13 mm to (129.2, 80.3)
- moved R1 3.13 mm to (130.6, 107.2)
- moved R2 3.13 mm to (120.5, 104.1)
- moved R3 3.13 mm to (120.5, 98.5)
- moved R4 3.13 mm to (120.5, 114.0)
Connections:
- J2 pad 12: unconnected-(J2-Pin_12-Pad12) -> Net-(J2-Pin_12)
Routing:
- net Net-(J2-Pin_12): track 0.00 -> 64.9 mm
- net /+3.3V: track 34.3 -> 50.0 mm
- net /39: track 28.2 -> 24.7 mm
Other:
- board size 45 x 50.5 mm -> 45 x 52.5 mm

Commit message: version
Parts:
- removed C1, C2, C3: 10n, Capacitor_THT:C_Disc_D4.3mm_W1.9mm_P5.00mm
- removed R2, R3, R4: 1M, Resistor_THT:R_Axial_DIN0207_L6.3mm_D2.5mm_P10.16mm_Horizontal
- added BT1: Battery_Cell, Connector_PinHeader_2.54mm:PinHeader_1x02_P2.54mm_Vertical, F.Cu at (129.3, 122.4)
- J4: value Conn_01x05_Socket -> Conn_01x04_Socket; footprint Connector_PinSocket_2.54mm:PinSocket_1x05_P2.54mm_Vertical -> Connector_PinSocket_2.54mm:PinSocket_1x04_P2.54mm_Vertical
- moved J3 6.73 mm to (118.6, 87.4), turned to 90 degrees
- moved J4 6.31 mm to (129.0, 86.6)
- moved R1 0.54 mm to (130.6, 106.7)
Connections:
- J1 pad 1: unconnected-(J1-Pin_1-Pad1) -> /SDA
- J2 pad 10: unconnected-(J2-Pin_10-Pad10) -> /SCL
- J4 pad 1: Net-(J4-Pin_1) -> /SDA
- J4 pad 2: Net-(J4-Pin_2) -> /SCL
- J4 pad 3: Net-(J4-Pin_3) -> GND
- J4 pad 4: Net-(J4-Pin_4) -> /+3.3V
Routing:
- net Net-(J4-Pin_2): track 37.6 -> 0.00 mm
- net Net-(J4-Pin_1): track 34.8 -> 0.00 mm
- net /SCL: track 0.00 -> 32.5 mm
- net Net-(J4-Pin_4): track 19.8 -> 0.00 mm
- net Net-(J4-Pin_3): track 16.7 -> 0.00 mm
- net /SDA: track 0.00 -> 9.76 mm
- net /35: track 7.12 -> 0.00 mm
- net /36: track 5.87 -> 0.00 mm
- net /34: track 5.76 -> 0.00 mm
- net /+5V: track 2.97 -> 6.64 mm
- net /39: track 24.7 -> 27.3 mm
- net /+3.3V: track 50.0 -> 48.2 mm
Other:
- board text added: "+"
- board text added: "+3.3V"
- board text added: "GND"
- board text added: "SCL"
- board text added: "SDA"

Commit message: 19/03
Parts:
- added D1: LED, LED_THT:LED_D3.0mm, F.Cu at (120.5, 121.0)
- added R2: 190, Resistor_THT:R_Axial_DIN0207_L6.3mm_D2.5mm_P10.16mm_Horizontal, F.Cu at (130.7, 113.8)
- J4: footprint Connector_PinSocket_2.54mm:PinSocket_1x04_P2.54mm_Vertical -> Connector_PinSocket_2.54mm:PinSocket_1x08_P2.54mm_Vertical
- moved R1 1.05 mm to (130.7, 107.7)
Connections:
- BT1 pad 1: /+5V -> /+3.3V
Routing:
- net /+3.3V: track 48.2 -> 56.1 mm
- net Net-(D1-A): track 0.00 -> 4.67 mm
- net /+5V: track 6.64 -> 2.97 mm
- net /39: track 27.3 -> 30.1 mm

Commit message: 01/04/25
Parts:
- added SW2: SW_DIP_x01, Button_Switch_THT:SW_slide-03_P5_THT, F.Cu at (121.6, 98.0)
- J4: value Conn_01x04_Socket -> Conn_01x08_Socket; footprint Connector_PinSocket_2.54mm:PinSocket_1x08_P2.54mm_Vertical -> Connector_PinHeader_2.54mm:PinHeader_1x08_P2.54mm_Vertical
- moved D1 1.26 mm to (120.5, 119.7)
Connections:
- BT1 pad 1: /+3.3V -> Net-(BT1-+)
- J4 pad 5: (no net) -> unconnected-(J4-Pin_5-Pad5)
- J4 pad 6: (no net) -> unconnected-(J4-Pin_6-Pad6)
- J4 pad 7: (no net) -> unconnected-(J4-Pin_7-Pad7)
- J4 pad 8: (no net) -> unconnected-(J4-Pin_8-Pad8)
Routing:
- net Net-(BT1-+): track 0.00 -> 22.6 mm
- net Net-(D1-A): track 4.67 -> 3.42 mm
Other:
- outline, holes or cut-outs redrawn
