File: carte_robo_main/Carte_main.kicad_sch (KiCad schematic)
At the start: 14 parts, among them J1 Conn_01x18_Pin, J2 Conn_01x18_Pin, J3 Conn_01x02_Socket, J4 Conn_01x05_Socket

Commit message: pcb done
Parts:
- C1, C2, C3: value 470n -> 10n; footprint (none) -> Capacitor_THT:C_Disc_D4.3mm_W1.9mm_P5.00mm
- C4, C5: footprint (none) -> Capacitor_THT:C_Disc_D4.3mm_W1.9mm_P5.00mm
- J3: footprint (none) -> Connector_PinHeader_2.54mm:PinHeader_1x02_P2.54mm_Vertical
- R1, R2, R3, R4: footprint (none) -> Resistor_THT:R_Axial_DIN0207_L6.3mm_D2.5mm_P10.16mm_Horizontal
Connections:
- net GND: now also C4.2, C5.2, J1.18 (Pin_18)
Changed lines of the file:
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@@
+	(wire
+		(pts
+			(xy 135.89 139.7) (xy 135.89 137.16)
+		)
+		(stroke
+			(width 0)
+			(type default)
+		)
+	)
 	(wire
 		(pts
@@
 			)
 		)
-		(property "Footprint" ""
+		(property "Footprint" "Resistor_THT:R_Axial_DIN0207_L6.3mm_D2.5mm_P10.16mm_Horizontal"
 			(at 58.42 88.9 0)
 			(effects
@@
 			)
 		)
-		(property "Footprint" ""
+		(property "Footprint" "Capacitor_THT:C_Disc_D4.3mm_W1.9mm_P5.00mm"
 			(at 135.89 128.27 0)
 			(effects
@@
 			)
 		)
-		(property "Footprint" ""
+		(property "Footprint" "Resistor_THT:R_Axial_DIN0207_L6.3mm_D2.5mm_P10.16mm_Horizontal"
 			(at 46.99 130.81 0)
 			(effects
@@
 			)
 		)
-		(property "Value" "470n"
+		(property "Value" "10n"
 			(at 57.15 106.6862 0)
 			(effects
@@
 			)
 		)
-		(property "Footprint" ""
+		(property "Footprint" "Capacitor_THT:C_Disc_D4.3mm_W1.9mm_P5.00mm"
 			(at 54.61 105.41 0)
 			(effects
@@
 			)
 		)
-		(property "Value" "470n"
+		(property "Value" "10n"
 			(at 74.93 106.6862 0)
 			(effects
@@
 			)
 		)
-		(property "Footprint" ""
+		(property "Footprint" "Capacitor_THT:C_Disc_D4.3mm_W1.9mm_P5.00mm"
 			(at 72.39 105.41 0)
 			(effects
@@
 				(path "/dbe09f27-eeb4-4ee6-a89f-2ca6fbf5bee0"
 					(reference "#PWR02")
+					(unit 1)
+				)
+			)
+		)
+	)
+	(symbol
+		(lib_id "power:GND")
+		(at 135.89 139.7 0)
+		(unit 1)
+		(exclude_from_sim no)
+		(in_bom yes)
+		(on_board yes)
+		(dnp no)
+		(fields_autoplaced yes)
+		(property "Reference" "#PWR03"
+			(at 135.89 146.05 0)
+			(effects
+				(font
+					(size 1.27 1.27)
+				)
+				(hide yes)
+			)
+		)
+		(property "Value" "GND"
+			(at 135.89 144.78 0)
+			(effects
+				(font
+					(size 1.27 1.27)
+				)
+			)
+		)
+		(property "Footprint" ""
+			(at 135.89 139.7 0)
+			(effects
+				(font
+					(size 1.27 1.27)
+				)
+				(hide yes)
+			)
+		)
+		(property "Datasheet" ""
+			(at 135.89 139.7 0)
+			(effects
+				(font
+					(size 1.27 1.27)
+				)
+				(hide yes)
+			)
+		)
+		(property "Description" "Power symbol creates a global label with name \"GND\" , ground"
+			(at 135.89 139.7 0)
+			(effects
+				(font
+					(size 1.27 1.27)
+				)
+				(hide yes)
+			)
+		)
+		(pin "1"
+		)
+		(instances
+			(project "Carte_main"
+				(path "/dbe09f27-eeb4-4ee6-a89f-2ca6fbf5bee0"
+					(reference "#PWR03")
 					(unit 1)
 				)
@@
 			)
 		)
-		(property "Footprint" ""
+		(property "Footprint" "Resistor_THT:R_Axial_DIN0207_L6.3mm_D2.5mm_P10.16mm_Horizontal"
 			(at 49.53 86.36 0)
 			(effects
@@
 			)
 		)
-		(property "Footprint" ""
+		(property "Footprint" "Connector_PinHeader_2.54mm:PinHeader_1x02_P2.54mm_Vertical"
 			(at 31.75 124.46 0)
 			(effects
@@
 			)
 		)
-		(property "Footprint" ""
+		(property "Footprint" "Resistor_THT:R_Axial_DIN0207_L6.3mm_D2.5mm_P10.16mm_Horizontal"
 			(at 67.31 91.44 0)
 			(effects
@@
 			)
 		)
-		(property "Value" "470n"
+		(property "Value" "10n"
 			(at 66.04 106.6862 0)
 			(effects
@@
 			)
 		)
-		(property "Footprint" ""
+		(property "Footprint" "Capacitor_THT:C_Disc_D4.3mm_W1.9mm_P5.00mm"
 			(at 63.5 105.41 0)
 			(effects
@@
 		(exclude_from_sim no)
 		(in_bom yes)
-		(on_board yes)
+		(on_board no)
 		(dnp no)
 		(fields_autoplaced yes)
@@
 			)
 		)
-		(property "Footprint" ""
+		(property "Footprint" "Capacitor_THT:C_Disc_D4.3mm_W1.9mm_P5.00mm"
 			(at 128.27 128.27 0)
 			(effects

Commit message: last update
Parts:
- added R5: 100k, Resistor_THT:R_Axial_DIN0207_L6.3mm_D2.5mm_P10.16mm_Horizontal, symbol GW_Passives:R_Small
- added SW1: SW_Push, Button_Switch_THT:SW_PUSH_6mm_H5mm, symbol GW_Mechanical:SW_Push
Connections:
- net +3.3V: now also SW1.1
- net GND: now also R5.1
- net at J2.12 (Pin_12): now also R5.2, SW1.2
- no-connect marks 24 -> 23

Commit message: version
Parts:
- removed C1, C2, C3: 10n, Capacitor_THT:C_Disc_D4.3mm_W1.9mm_P5.00mm, symbol GW_Passives:C_Small
- removed J4: Conn_01x05_Socket, Connector_PinSocket_2.54mm:PinSocket_1x05_P2.54mm_Vertical, symbol Connector:Conn_01x05_Socket
- removed R2, R3, R4: 1M, Resistor_THT:R_Axial_DIN0207_L6.3mm_D2.5mm_P10.16mm_Horizontal, symbol GW_Passives:R_Small
- added J4: Conn_01x04_Socket, Connector_PinSocket_2.54mm:PinSocket_1x04_P2.54mm_Vertical, symbol Connector:Conn_01x04_Socket
- BT1: footprint (none) -> Connector_PinHeader_2.54mm:PinHeader_1x02_P2.54mm_Vertical
Connections:
- net +3.3V: now also J4.4 (Pin_4)
- net GND: now also J4.3 (Pin_3)
- net SDA: now reaches J1.1 (Pin_1)
- net SDA: now also J4.1 (Pin_1)
- net SCL: now reaches J2.10 (Pin_10)
- net SCL: now also J4.2 (Pin_2)
- no-connect marks 23 -> 21
Other:
- moved on the sheet: BT1, J3, R1

Commit message: 19/03
Parts:
- added D1: LED, LED_THT:LED_D3.0mm, symbol Device:LED
- added R2: 190, Resistor_THT:R_Axial_DIN0207_L6.3mm_D2.5mm_P10.16mm_Horizontal, symbol GW_Passives:R_Small
- J4: footprint Connector_PinSocket_2.54mm:PinSocket_1x04_P2.54mm_Vertical -> Connector_PinSocket_2.54mm:PinSocket_1x08_P2.54mm_Vertical
Connections:
- net +3.3V: now also BT1.1 (+), R2.1
- net +5V: no longer BT1.1 (+)
- net GND: now also D1.1 (K)
- new net: D1.2 (A), R2.2
Other:
- moved on the sheet: BT1, J3, J4, R1

Commit message: 01/04/25
Parts:
- removed J4: Conn_01x04_Socket, Connector_PinSocket_2.54mm:PinSocket_1x08_P2.54mm_Vertical, symbol Connector:Conn_01x04_Socket
- added J4: Conn_01x08_Socket, Connector_PinHeader_2.54mm:PinHeader_1x08_P2.54mm_Vertical, symbol Connector:Conn_01x08_Socket
- added SW2: SW_DIP_x01, Button_Switch_THT:SW_slide-03_P5_THT, symbol Switch:SW_DIP_x01
Connections:
- net +3.3V: now also J4.4 (Pin_4), SW2.2; no longer BT1.1 (+)
- net GND: now also J4.3 (Pin_3)
- net SCL: now also J4.2 (Pin_2)
- net SDA: now also J4.1 (Pin_1)
- new net: BT1.1 (+), SW2.1
- no-connect marks 21 -> 25
Other:
- moved on the sheet: BT1
Changed lines of the file:
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@@
+	)
+	(junction
+		(at 100.33 105.41)
+		(diameter 0)
+		(color 0 0 0 0)
 	)
 	(junction
@@
 		(color 0 0 0 0)
 	)
-	(junction
-		(at 100.33 105.41)
-		(diameter 0)
-		(color 0 0 0 0)
-	)
 	(no_connect
 		(at 172.72 113.03)
@@
 	)
 	(no_connect
+		(at 93.98 55.88)
+	)
+	(no_connect
 		(at 172.72 115.57)
 	)
@@
 	)
 	(no_connect
+		(at 93.98 58.42)
+	)
+	(no_connect
 		(at 140.97 90.17)
 	)
 	(no_connect
+		(at 93.98 63.5)
+	)
+	(no_connect
 		(at 172.72 80.01)
 	)
@@
 	)
 	(no_connect
+		(at 93.98 60.96)
+	)
+	(no_connect
 		(at 140.97 95.25)
 	)
@@
 	(wire
 		(pts
-			(xy 67.31 151.13) (xy 67.31 148.59)
-		)
-		(stroke
-			(width 0)
-			(type default)
-		)
-	)
-	(wire
-		(pts
 			(xy 93.98 66.04) (xy 100.33 66.04)
 		)
@@
 	(wire
 		(pts
+			(xy 67.31 148.59) (xy 67.31 152.4)
+		)
+		(stroke
+			(width 0)
+			(type default)
+		)
+	)
+	(wire
+		(pts
 			(xy 100.33 105.41) (xy 100.33 109.22)
 		)
@@
 	(wire
 		(pts
-			(xy 67.31 158.75) (xy 67.31 166.37)
+			(xy 67.31 179.07) (xy 67.31 187.96)
 		)
 		(stroke
@@
 		(pts
 			(xy 201.93 92.71) (xy 190.5 92.71)
+		)
+		(stroke
+			(width 0)
+			(type default)
+		)
+	)
+	(wire
+		(pts
+			(xy 67.31 167.64) (xy 67.31 171.45)
 		)
 		(stroke
@@
 				(path "/dbe09f27-eeb4-4ee6-a89f-2ca6fbf5bee0"
 					(reference "J1")
+					(unit 1)
+				)
+			)
+		)
+	)
+	(symbol
+		(lib_id "Switch:SW_DIP_x01")
+		(at 67.31 160.02 90)
+		(unit 1)
+		(exclude_from_sim no)
+		(in_bom yes)
+		(on_board yes)
+		(dnp no)
+		(fields_autoplaced yes)
+		(property "Reference" "SW2"
+			(at 71.12 158.7499 90)
+			(effects
+				(font
+					(size 1.27 1.27)
+				)
+				(justify right)
+			)
+		)
+		(property "Value" "SW_DIP_x01"
+			(at 71.12 161.2899 90)
+			(effects
+				(font
+					(size 1.27 1.27)
+				)
+				(justify right)
+			)
+		)
+		(property "Footprint" "Button_Switch_THT:SW_slide-03_P5_THT"
+			(at 67.31 160.02 0)
+			(effects
+				(font
+					(size 1.27 1.27)
+				)
+				(hide yes)
+			)
+		)
+		(property "Datasheet" "~"
+			(at 67.31 160.02 0)
+			(effects
+				(font
+					(size 1.27 1.27)
+				)
+				(hide yes)
+			)
+		)
+		(property "Description" "1x DIP Switch, Single Pole Single Throw (SPST) switch, small symbol"
+			(at 67.31 160.02 0)
+			(effects
+				(font
+					(size 1.27 1.27)
+				)
+				(hide yes)
+			)
+		)
+		(pin "2"
+		)
+		(pin "1"
+		)
+		(instances
+			(project "Carte_main"
+				(path "/dbe09f27-eeb4-4ee6-a89f-2ca6fbf5bee0"
+					(reference "SW2")
 					(unit 1)
 				)
@@
 	(symbol
 		(lib_id "power:GND")
-		(at 67.31 166.37 0)
+		(at 67.31 187.96 0)
 		(unit 1)
 		(exclude_from_sim no)
@@
 		(fields_autoplaced yes)
 		(property "Reference" "#PWR02"
-			(at 67.31 172.72 0)
+			(at 67.31 194.31 0)
 			(effects
 				(font
@@
 		)
 		(property "Value" "GND"
-			(at 67.31 171.45 0)
+			(at 67.31 193.04 0)
 			(effects
 				(font
@@
 		)
 		(property "Footprint" ""
-			(at 67.31 166.37 0)
+			(at 67.31 187.96 0)
 			(effects
 				(font
@@
 		)
 		(property "Datasheet" ""
-			(at 67.31 166.37 0)
+			(at 67.31 187.96 0)
 			(effects
 				(font
@@
 		)
 		(property "Description" "Power symbol creates a global label with name \"GND\" , ground"
-			(at 67.31 166.37 0)
+			(at 67.31 187.96 0)
 			(effects
 				(font
@@
 				(path "/dbe09f27-eeb4-4ee6-a89f-2ca6fbf5bee0"
 					(reference "#PWR02")
+					(unit 1)
+				)
+			)
+		)
+	)
+	(symbol
+		(lib_id "Connector:Conn_01x08_Socket")
+		(at 88.9 66.04 180)
+		(unit 1)
+		(exclude_from_sim no)
+		(in_bom yes)
+		(on_board yes)
+		(dnp no)
+		(fields_autoplaced yes)
+		(property "Reference" "J4"
+			(at 89.535 50.8 0)
+			(effects
+				(font
+					(size 1.27 1.27)
+				)
+			)
+		)
+		(property "Value" "Conn_01x08_Socket"
+			(at 89.535 53.34 0)
+			(effects
+				(font
+					(size 1.27 1.27)
+				)
+			)
+		)
+		(property "Footprint" "Connector_PinHeader_2.54mm:PinHeader_1x08_P2.54mm_Vertical"
+			(at 88.9 66.04 0)
+			(effects
+				(font
+					(size 1.27 1.27)
+				)
+				(hide yes)
+			)
+		)
+		(property "Datasheet" "~"
+			(at 88.9 66.04 0)
+			(effects
+				(font
+					(size 1.27 1.27)
+				)
+				(hide yes)
+			)
+		)
+		(property "Description" "Generic connector, single row, 01x08, script generated"
+			(at 88.9 66.04 0)
+			(effects
+				(font
+					(size 1.27 1.27)
+				)
+				(hide yes)
+			)
+		)
+		(pin "2"
+		)
+		(pin "4"
+		)
+		(pin "6"
+		)
+		(pin "7"
+		)
+		(pin "5"
+		)
+		(pin "3"
+		)
+		(pin "8"
+		)
+		(pin "1"
+		)
+		(instances
+			(project "Carte_main"
+				(path "/dbe09f27-eeb4-4ee6-a89f-2ca6fbf5bee0"
+					(reference "J4")
 					(unit 1)
 				)
@@
 				(path "/dbe09f27-eeb4-4ee6-a89f-2ca6fbf5bee0"
 					(reference "J3")
-					(unit 1)
-				)
-			)
-		)
-	)
-	(symbol
-		(lib_id "Connector:Conn_01x04_Socket")
-		(at 88.9 71.12 180)
-		(unit 1)
-		(exclude_from_sim no)
-		(in_bom yes)
-		(on_board yes)
-		(dnp no)
-		(fields_autoplaced yes)
-		(property "Reference" "J4"
-			(at 89.535 60.96 0)
-			(effects
-				(font
-					(size 1.27 1.27)
-				)
-			)
-		)
-		(property "Value" "Conn_01x04_Socket"
-			(at 89.535 63.5 0)
-			(effects
-				(font
-					(size 1.27 1.27)
-				)
-			)
-		)
-		(property "Footprint" "Connector_PinSocket_2.54mm:PinSocket_1x08_P2.54mm_Vertical"
-			(at 88.9 71.12 0)
-			(effects
-				(font
-					(size 1.27 1.27)
-				)
-				(hide yes)
-			)
-		)
-		(property "Datasheet" "~"
-			(at 88.9 71.12 0)
-			(effects
-				(font
-					(size 1.27 1.27)
-				)
-				(hide yes)
-			)
-		)
-		(property "Description" "Generic connector, single row, 01x04, script generated"
-			(at 88.9 71.12 0)
-			(effects
-				(font
-					(size 1.27 1.27)
-				)
-				(hide yes)
-			)
-		)
-		(pin "1"
-		)
-		(pin "4"
-		)
-		(pin "2"
-		)
-		(pin "3"
-		)
-		(instances
-			(project "Carte_main"
-				(path "/dbe09f27-eeb4-4ee6-a89f-2ca6fbf5bee0"
-					(reference "J4")
 					(unit 1)
 				)
@@
 	(symbol
 		(lib_id "GW_Mechanical:Battery_Cell")
-		(at 67.31 156.21 0)
+		(at 67.31 176.53 0)
 		(unit 1)
 		(exclude_from_sim no)
@@
 		(fields_autoplaced yes)
 		(property "Reference" "BT1"
-			(at 71.12 153.0984 0)
+			(at 71.12 173.4184 0)
 			(effects
 				(font
@@
 		)
 		(property "Value" "Battery_Cell"
-			(at 71.12 155.6384 0)
+			(at 71.12 175.9584 0)
 			(effects
 				(font
@@
 		)
 		(property "Footprint" "Connector_PinHeader_2.54mm:PinHeader_1x02_P2.54mm_Vertical"
-			(at 67.31 154.686 90)
+			(at 67.31 175.006 90)
 			(effects
 				(font
@@
 		)
 		(property "Datasheet" "~"
-			(at 67.31 154.686 90)
+			(at 67.31 175.006 90)
 			(effects
 				(font
@@
 		)
 		(property "Description" "Single-cell battery"
-			(at 67.31 156.21 0)
+			(at 67.31 176.53 0)
 			(effects
 				(font
@@
 		)
 		(property "Manufacturer" ""
-			(at 67.31 156.21 0)
-			(effects
-				(font
+			(at 67.31 176.53 0)
+			(effects
+				(font
